File: PCB/PCB.kicad_pcb (KiCad board)
At the start: 2 copper layers, 29 parts, among them J1 TFT Display, J10 VBUS, J11 3V3_EN, J12 Rotary Encoder, J13 RE Button, J14 Green Button, J15 Red Button, J16 ADC_VREF, J17 GPIO28, J18 AGND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

Commit message: Finished PCB, Last commit before moving to Bradley Org
Parts:
- added G***: LOGO, CarImage, F.Cu at (111.5, 133.0)
- added REF**: MountingHole_3.2mm_M3_DIN965_Pad_TopBottom, MountingHole:MountingHole_3.2mm_M3_DIN965_Pad_TopBottom, F.Cu at (102.0, 59.5)
- added REF**: MountingHole_3.2mm_M3_DIN965_Pad_TopBottom, MountingHole:MountingHole_3.2mm_M3_DIN965_Pad_TopBottom, F.Cu at (163.0, 132.5)
- added REF**: MountingHole_3.2mm_M3_DIN965_Pad_TopBottom, MountingHole:MountingHole_3.2mm_M3_DIN965_Pad_TopBottom, F.Cu at (102.0, 132.5)
- added REF**: MountingHole_3.2mm_M3_DIN965_Pad_TopBottom, MountingHole:MountingHole_3.2mm_M3_DIN965_Pad_TopBottom, F.Cu at (163.0, 59.5)
- moved J9 11.2 mm to (164.0, 74.0)
- moved J6 5.22 mm to (107.5, 107.8)
- moved J3 2.54 mm to (154.5, 64.4)
Routing:
- net Net-(J1-Pin_5): track 21.9 -> 46.9 mm
- net Net-(J15-Pin_2): track 27.3 -> 17.2 mm
- net Net-(J1-Pin_6): track 28.5 -> 19.5 mm
- net Net-(J2-Pin_8): track 81.4 -> 89.6 mm
- net Net-(J6-Pin_6): track 38.5 -> 46.5 mm
- net Net-(J1-Pin_11): track 24.3 -> 17.4 mm
- net Net-(J4-Pin_4): track 34.9 -> 29.3 mm
- net Net-(J1-Pin_1): track 120.7 -> 115.3 mm
- net Net-(J1-Pin_4): track 23.0 -> 18.5 mm
- net Net-(J12-Pin_3): track 22.1 -> 19.5 mm
- net Net-(J13-Pin_2): track 22.8 -> 20.8 mm
- net Net-(J2-Pin_4): track 31.4 -> 32.9 mm
- net Net-(J9-Pin_2): track 6.21 -> 6.93 mm
- net Net-(J4-Pin_1): track 25.6 -> 26.1 mm
Other:
- board outline added: 70 x 82 mm
- board text added: "DC"
- board text added: "RST"
- board text added: "Superyardage Controller"
